File: Flipper_PCB/Flipper_PCB.sch (KiCad schematic (older format))
At the start: 11 parts, among them J1 Conn_01x16

Commit message: pcb ready
Parts:
- added Btn1: Screw_Terminal_01x02, TerminalBlock:TerminalBlock_bornier-2_P5.08mm, symbol Connector:Screw_Terminal_01x02
- 12V1, 5V1, GND1, GND2: footprint (none) -> Connector_PinHeader_2.54mm:PinHeader_1x01_P2.54mm_Vertical
- ESP32_L1: renamed from Left1; footprint Connector_PinHeader_2.54mm:PinHeader_1x19_P2.54mm_Vertical -> Connector_PinSocket_2.54mm:PinSocket_1x19_P2.54mm_Vertical
- ESP32_R1: renamed from Right1; footprint Connector_PinHeader_2.54mm:PinHeader_1x19_P2.54mm_Vertical -> Connector_PinSocket_2.54mm:PinSocket_1x19_P2.54mm_Vertical
- MusicMaker_Left1: footprint Connector_PinHeader_2.54mm:PinHeader_1x12_P2.54mm_Vertical -> Connector_PinSocket_2.54mm:PinSocket_1x12_P2.54mm_Vertical
- MusicMaker_Right1: renamed from J1; footprint Connector_PinHeader_2.54mm:PinHeader_1x16_P2.54mm_Vertical -> Connector_PinSocket_2.54mm:PinSocket_1x16_P2.54mm_Vertical
- SERIAL1: footprint Connector_PinHeader_2.54mm:PinHeader_1x04_P2.54mm_Vertical -> Connector_PinSocket_2.54mm:PinSocket_1x04_P2.54mm_Vertical
Connections:
- net GND: now reaches ESP32_R1.1 (Pin_1)
- net GND: now also GND2.1 (Pin_1), MusicMaker_Right1.13 (Pin_13), SERIAL1.4 (Pin_4), ServoData-GND1.2 (Pin_2), Btn1.2 (Pin_2)
- net BTN: now reaches ESP32_R1.12 (Pin_12)
- net BTN: now also Btn1.1 (Pin_1)
- net DREQ: now reaches ESP32_R1.16 (Pin_16)
- net DREQ: now also MusicMaker_Left1.5 (Pin_5)
- net MOSI: now reaches ESP32_R1.2 (Pin_2)
- net MOSI: now also MusicMaker_Right1.5 (Pin_5)
- net MISO: now reaches ESP32_R1.8 (Pin_8)
- net MISO: now also MusicMaker_Right1.4 (Pin_4)
- net SCK: now reaches ESP32_R1.9 (Pin_9)
- net SCK: now also MusicMaker_Right1.6 (Pin_6)
- net 3V3: now reaches ESP32_L1.1 (Pin_1)
- net 3V3: now also MusicMaker_Right1.15 (Pin_15)
- net SDCS: now reaches ESP32_L1.12 (Pin_12)
- net SDCS: now also MusicMaker_Left1.3 (Pin_3)
- net ServoData: now reaches ESP32_L1.13 (Pin_13)
- net ServoData: now also ServoData-GND1.1 (Pin_1)
- net RX: now reaches ESP32_L1.17 (Pin_17)
- net RX: now also SERIAL1.3 (Pin_3)
- net +5V: now reaches ESP32_L1.19 (Pin_19)
- net +5V: now also 5V1.1 (Pin_1), SERIAL1.1 (Pin_1)
- net MP3CS: now reaches ESP32_L1.7 (Pin_7)
- net MP3CS: now also MusicMaker_Left1.4 (Pin_4)
- net XDCS: now reaches ESP32_L1.8 (Pin_8)
- net XDCS: now also MusicMaker_Left1.6 (Pin_6)
- net at 12V-GND1.1 (Pin_1): now also 12V1.1 (Pin_1)
- net at 12V-GND1.2 (Pin_2): now also GND1.1 (Pin_1)
Other:
- note added: "12V -> 5V Converter"
- note added: "3V3"
- moved on the sheet: ESP32_L1
Changed lines of the file:
@@
 $EndDescr
 $Comp
-L Connector_Generic:ESP32_DevKitC_Right Right1
-U 1 1 5DCD3C29
-P 6450 2750
-F 0 "Right1" H 6368 3867 50  0000 C CNN
-F 1 "ESP32_DevKitC_Right" H 6368 3776 50  0000 C CNN
-F 2 "Connector_PinHeader_2.54mm:PinHeader_1x19_P2.54mm_Vertical" H 6450 1700 50  0001 C CNN
-F 3 "" H 6450 1700 50  0001 C CNN
-	1    6450 2750
-	-1   0    0    -1
-$EndComp
-$Comp
-L Connector_Generic:ESP32_DevKitC_Left Left1
+L Connector_Generic:ESP32_DevKitC_Left ESP32_L1
 U 1 1 5DCED2C2
-P 5700 2800
-F 0 "Left1" H 5780 2892 50  0000 C CNN
-F 1 "ESP32_DevKitC_Left" H 5780 2801 50  0000 C CNN
-F 2 "Connector_PinHeader_2.54mm:PinHeader_1x19_P2.54mm_Vertical" H 5700 1800 50  0001 C CNN
-F 3 "" H 5700 1800 50  0001 C CNN
-	1    5700 2800
+P 5750 2800
+F 0 "ESP32_L1" H 5830 2892 50  0000 C CNN
+F 1 "ESP32_DevKitC_Left" H 5830 2801 50  0000 C CNN
+F 2 "Connector_PinSocket_2.54mm:PinSocket_1x19_P2.54mm_Vertical" H 5750 1800 50  0001 C CNN
+F 3 "" H 5750 1800 50  0001 C CNN
+	1    5750 2800
 	1    0    0    -1
 $EndComp
@@
 F 0 "MusicMaker_Left1" H 3680 2342 50  0001 L CNN
 F 1 "Conn_01x12" H 3680 2251 50  0001 L CNN
-F 2 "Connector_PinHeader_2.54mm:PinHeader_1x12_P2.54mm_Vertical" H 3600 2350 50  0001 C CNN
+F 2 "Connector_PinSocket_2.54mm:PinSocket_1x12_P2.54mm_Vertical" H 3600 2350 50  0001 C CNN
 F 3 "~" H 3600 2350 50  0001 C CNN
 	1    3600 2350
@@
 F 0 "SERIAL1" H 7680 1892 50  0001 L CNN
 F 1 "Conn_01x04" H 7680 1801 50  0001 L CNN
-F 2 "Connector_PinHeader_2.54mm:PinHeader_1x04_P2.54mm_Vertical" H 7600 1900 50  0001 C CNN
+F 2 "Connector_PinSocket_2.54mm:PinSocket_1x04_P2.54mm_Vertical" H 7600 1900 50  0001 C CNN
 F 3 "~" H 7600 1900 50  0001 C CNN
 	1    7600 1900
@@
 U 1 1 5DD14FF9
 P 2350 950
-F 0 "12V1" H 2268 817 50  0000 C CNN
+F 0 "12V1" H 2268 817 50  0001 C CNN
 F 1 "Conn_01x01" H 2430 901 50  0001 L CNN
-F 2 "" H 2350 950 50  0001 C CNN
+F 2 "Connector_PinHeader_2.54mm:PinHeader_1x01_P2.54mm_Vertical" H 2350 950 50  0001 C CNN
 F 3 "~" H 2350 950 50  0001 C CNN
 	1    2350 950
@@
 U 1 1 5DD16AAC
 P 2350 1250
-F 0 "GND1" H 2268 1117 50  0000 C CNN
+F 0 "GND1" H 2268 1117 50  0001 C CNN
 F 1 "Conn_01x01" H 2430 1201 50  0001 L CNN
-F 2 "" H 2350 1250 50  0001 C CNN
+F 2 "Connector_PinHeader_2.54mm:PinHeader_1x01_P2.54mm_Vertical" H 2350 1250 50  0001 C CNN
 F 3 "~" H 2350 1250 50  0001 C CNN
 	1    2350 1250
@@
 L Connector_Generic:Conn_01x01 5V1
 U 1 1 5DD16FF6
-P 2850 950
-F 0 "5V1" H 2768 817 50  0000 C CNN
-F 1 "Conn_01x01" H 2930 901 50  0001 L CNN
-F 2 "" H 2850 950 50  0001 C CNN
-F 3 "~" H 2850 950 50  0001 C CNN
-	1    2850 950
-	1    0    0    1
+P 2550 950
+F 0 "5V1" H 2468 817 50  0001 C CNN
+F 1 "Conn_01x01" H 2630 901 50  0001 L CNN
+F 2 "Connector_PinHeader_2.54mm:PinHeader_1x01_P2.54mm_Vertical" H 2550 950 50  0001 C CNN
+F 3 "~" H 2550 950 50  0001 C CNN
+	1    2550 950
+	-1   0    0    -1
 $EndComp
 $Comp
 L Connector_Generic:Conn_01x01 GND2
 U 1 1 5DD172E1
-P 2850 1250
-F 0 "GND2" H 2768 1117 50  0000 C CNN
-F 1 "Conn_01x01" H 2930 1201 50  0001 L CNN
-F 2 "" H 2850 1250 50  0001 C CNN
-F 3 "~" H 2850 1250 50  0001 C CNN
-	1    2850 1250
-	1    0    0    1
+P 2550 1250
+F 0 "GND2" H 2468 1117 50  0001 C CNN
+F 1 "Conn_01x01" H 2630 1201 50  0001 L CNN
+F 2 "Connector_PinHeader_2.54mm:PinHeader_1x01_P2.54mm_Vertical" H 2550 1250 50  0001 C CNN
+F 3 "~" H 2550 1250 50  0001 C CNN
+	1    2550 1250
+	-1   0    0    -1
 $EndComp
 $Comp
@@
 $EndComp
 $Comp
-L Connector_Generic:Conn_01x16 J1
+L Connector_Generic:Conn_01x16 MusicMaker_Right1
 U 1 1 5DD1DD42
 P 4350 2550
-F 0 "J1" H 4268 3467 50  0001 C CNN
+F 0 "MusicMaker_Right1" H 4268 3467 50  0001 C CNN
 F 1 "Conn_01x16" H 4268 3376 50  0001 C CNN
-F 2 "Connector_PinHeader_2.54mm:PinHeader_1x16_P2.54mm_Vertical" H 4350 2550 50  0001 C CNN
+F 2 "Connector_PinSocket_2.54mm:PinSocket_1x16_P2.54mm_Vertical" H 4350 2550 50  0001 C CNN
 F 3 "~" H 4350 2550 50  0001 C CNN
 	1    4350 2550
 	-1   0    0    -1
 $EndComp
+Wire Wire Line
+	1450 950  2150 950
+Wire Wire Line
+	1450 1050 2150 1250
+$Comp
+L power:+5V #PWR0101
+U 1 1 5DCD9FF6
+P 2750 950
+F 0 "#PWR0101" H 2750 800 50  0001 C CNN
+F 1 "+5V" V 2765 1078 50  0000 L CNN
+F 2 "" H 2750 950 50  0001 C CNN
+F 3 "" H 2750 950 50  0001 C CNN
+	1    2750 950
+	0    1    1    0
+$EndComp
+$Comp
+L power:GND #PWR0102
+U 1 1 5DCDAB77
+P 2750 1250
+F 0 "#PWR0102" H 2750 1000 50  0001 C CNN
+F 1 "GND" V 2755 1122 50  0000 R CNN
+F 2 "" H 2750 1250 50  0001 C CNN
+F 3 "" H 2750 1250 50  0001 C CNN
+	1    2750 1250
+	0    -1   -1   0
+$EndComp
+Text Notes 2150 800  0    50   ~ 0
+12V -> 5V Converter
+Text Notes 4150 3250 0    50   ~ 0
+3V3
+Text Notes 4150 3050 0    50   ~ 0
+GND
+$Comp
+L power:+5V #PWR0103
+U 1 1 5DCDBF8C
+P 5500 3650
+F 0 "#PWR0103" H 5500 3500 50  0001 C CNN
+F 1 "+5V" V 5515 3778 50  0000 L CNN
+F 2 "" H 5500 3650 50  0001 C CNN
+F 3 "" H 5500 3650 50  0001 C CNN
+	1    5500 3650
+	0    -1   -1   0
+$EndComp
+$Comp
+L power:GND #PWR0104
+U 1 1 5DCDCAFA
+P 4550 3050
+F 0 "#PWR0104" H 4550 2800 50  0001 C CNN
+F 1 "GND" V 4555 2922 50  0000 R CNN
+F 2 "" H 4550 3050 50  0001 C CNN
+F 3 "" H 4550 3050 50  0001 C CNN
+	1    4550 3050
+	0    -1   -1   0
+$EndComp
+$Comp
+L power:GND #PWR0105
+U 1 1 5DCDDD08
+P 7400 2650
+F 0 "#PWR0105" H 7400 2400 50  0001 C CNN
+F 1 "GND" H 7405 2477 50  0000 C CNN
+F 2 "" H 7400 2650 50  0001 C CNN
+F 3 "" H 7400 2650 50  0001 C CNN
+	1    7400 2650
+	1    0    0    -1
+$EndComp
+$Comp
+L power:GND #PWR0106
+U 1 1 5DCDE90D
+P 7400 2100
+F 0 "#PWR0106" H 7400 1850 50  0001 C CNN
+F 1 "GND" H 7405 1927 50  0000 C CNN
+F 2 "" H 7400 2100 50  0001 C CNN
+F 3 "" H 7400 2100 50  0001 C CNN
+	1    7400 2100
+	1    0    0    -1
+$EndComp
+$Comp
+L power:+5V #PWR0107
+U 1 1 5DCDED2C
+P 7400 1800
+F 0 "#PWR0107" H 7400 1650 50  0001 C CNN
+F 1 "+5V" H 7415 1973 50  0000 C CNN
+F 2 "" H 7400 1800 50  0001 C CNN
+F 3 "" H 7400 1800 50  0001 C CNN
+	1    7400 1800
+	1    0    0    -1
+$EndComp
+Text GLabel 3400 2050 0    50   Input ~ 0
+SDCS
+Text GLabel 3400 2150 0    50   Input ~ 0
+MP3CS
+Text GLabel 3400 2250 0    50   Input ~ 0
+DREQ
+Text GLabel 3400 2350 0    50   Input ~ 0
+XDCS
+Text GLabel 4550 2150 2    50   Input ~ 0
+MISO
+Text GLabel 4550 2250 2    50   Input ~ 0
+MOSI
+Text GLabel 4550 2350 2    50   Input ~ 0
+SCK
+Text GLabel 5500 3450 0    50   Input ~ 0
+RX
+Text GLabel 7400 2000 0    50   Input ~ 0
+RX
+Text GLabel 5500 3050 0    50   Input ~ 0
+ServoData
+Text GLabel 5500 2950 0    50   Input ~ 0
+SDCS
+Text GLabel 5500 2450 0    50   Input ~ 0
+MP3CS
+Text GLabel 5500 2550 0    50   Input ~ 0
+XDCS
+Text GLabel 4550 3250 2    50   Input ~ 0
+3V3
+Text GLabel 5500 1850 0    50   Input ~ 0
+3V3
+Text GLabel 6650 2650 2    50   Input ~ 0
+SCK
+Text GLabel 6650 1950 2    50   Input ~ 0
+MOSI
+Text GLabel 6650 2550 2    50   Input ~ 0
+MISO
+Text GLabel 6650 3350 2    50   Input ~ 0
+DREQ
+Text GLabel 7400 2550 0    50   Input ~ 0
+ServoData
+$Comp
+L power:GND #PWR0109
+U 1 1 5DCDD9CF
+P 6650 1850
+F 0 "#PWR0109" H 6650 1600 50  0001 C CNN
+F 1 "GND" V 6655 1722 50  0000 R CNN
+F 2 "" H 6650 1850 50  0001 C CNN
+F 3 "" H 6650 1850 50  0001 C CNN
+	1    6650 1850
+	0    -1   -1   0
+$EndComp
+$Comp
+L Connector_Generic:ESP32_DevKitC_Right ESP32_R1
+U 1 1 5DCD3C29
+P 6450 2750
+F 0 "ESP32_R1" H 6368 3867 50  0000 C CNN
+F 1 "ESP32_DevKitC_Right" H 6368 3776 50  0000 C CNN
+F 2 "Connector_PinSocket_2.54mm:PinSocket_1x19_P2.54mm_Vertical" H 6450 1700 50  0001 C CNN
+F 3 "" H 6450 1700 50  0001 C CNN
+	1    6450 2750
+	-1   0    0    -1
+$EndComp
+$Comp
+L Connector:Screw_Terminal_01x02 Btn1
+U 1 1 5DCE5196
+P 7600 3100
+F 0 "Btn1" H 7680 3092 50  0000 L CNN
+F 1 "Screw_Terminal_01x02" H 7680 3001 50  0000 L CNN
+F 2 "TerminalBlock:TerminalBlock_bornier-2_P5.08mm" H 7600 3100 50  0001 C CNN
+F 3 "~" H 7600 3100 50  0001 C CNN
+	1    7600 3100
+	1    0    0    -1
+$EndComp
+$Comp
+L power:GND #PWR0108
+U 1 1 5DCE519C
+P 7400 3200
+F 0 "#PWR0108" H 7400 2950 50  0001 C CNN
+F 1 "GND" H 7405 3027 50  0000 C CNN
+F 2 "" H 7400 3200 50  0001 C CNN
+F 3 "" H 7400 3200 50  0001 C CNN
+	1    7400 3200
+	1    0    0    -1
+$EndComp
+Text GLabel 7400 3100 0    50   Input ~ 0
+BTN
+Text GLabel 6650 2950 2    50   Input ~ 0
+BTN
 $EndSCHEMATC
