File: Flipper_PCB/Flipper_PCB.kicad_pcb (KiCad board)
At the start: 2 copper layers, 134.6 x 58.4 mm, 14 parts, among them M4 MountingHole_4.3mm_M4

Commit message: ds
Parts:
- added M3: MountingHole_3.2mm_M3, MountingHole:MountingHole_3.2mm_M3, F.Cu at (151.1, 80.0)
- moved 12V1 10.2 mm to (193.0, 76.2)
- moved 5V1 10.2 mm to (193.0, 61.0)
- moved GND1 10.2 mm to (182.9, 76.2)
- moved GND2 10.2 mm to (182.9, 61.0)
- moved ServoData-GND1 5.08 mm to (172.7, 91.4), turned to 180 degrees
- moved 12V-GND1 5.08 mm to (193.0, 91.4), turned to 180 degrees
Routing:
- net +5V: track 120.5 -> 133.5 mm
- net ServoData: track 79.0 -> 85.6 mm
- net Net-(12V-GND1-Pad2): track 15.2 -> 18.4 mm
- net Net-(12V-GND1-Pad1): track 18.4 -> 15.2 mm
Other:
- board text added: "FAITES VOS JEUX !"
Changed lines of the file:
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@@
   (general
     (thickness 1.6)
-    (drawings 28)
-    (tracks 79)
+    (drawings 29)
+    (tracks 81)
     (zones 0)
-    (modules 14)
+    (modules 15)
     (nets 16)
   )
@@
     (add_net XDCS)
   )
+  (module MountingHole:MountingHole_3.2mm_M3 (layer F.Cu)
+    (at 151.13 80.01)
+    (descr "Mounting Hole 3.2mm, no annular, M3")
+    (tags "mounting hole 3.2mm no annular m3")
+    (attr virtual)
+    (fp_text reference M3 (at 0 -4.2) (layer F.SilkS)
+      (effects (font (size 1 1) (thickness 0.15)))
+    )
+    (fp_text value MountingHole_3.2mm_M3 (at 0 4.2) (layer F.Fab)
+      (effects (font (size 1 1) (thickness 0.15)))
+    )
+    (fp_circle (center 0 0) (end 3.45 0) (layer F.CrtYd) (width 0.05))
+    (fp_circle (center 0 0) (end 3.2 0) (layer Cmts.User) (width 0.15))
+    (fp_text user %R (at 0.3 0) (layer F.Fab)
+      (effects (font (size 1 1) (thickness 0.15)))
+    )
+    (pad 1 np_thru_hole circle (at 0 0) (size 3.2 3.2) (drill 3.2) (layers *.Cu *.Mask))
+  )
   (module MountingHole:MountingHole_4.3mm_M4 (layer F.Cu)
     (at 68.58 96.52)
@@
   )
   (module Connector_PinHeader_2.54mm:PinHeader_1x01_P2.54mm_Vertical (layer F.Cu)
-    (at 182.88 76.2 90)
+    (at 193.04 76.2 90)
     (descr "Through hole straight pin header, 1x01, 2.54mm pitch, single row")
     (tags "Through hole pin header THT 1x01 2.54mm single row")
@@
   )
   (module TerminalBlock:TerminalBlock_bornier-2_P5.08mm (layer F.Cu)
-    (at 187.96 91.44)
+    (at 193.04 91.44 180)
     (descr "simple 2-pin terminal block, pitch 5.08mm, revamped version of bornier2")
     (tags "terminal block bornier2")
@@
       (effects (font (size 1 1) (thickness 0.15)))
     )
-    (pad 2 thru_hole circle (at 5.08 0) (size 3 3) (drill 1.52) (layers *.Cu *.Mask)
+    (pad 2 thru_hole circle (at 5.08 0 180) (size 3 3) (drill 1.52) (layers *.Cu *.Mask)
       (net 2 "Net-(12V-GND1-Pad2)"))
-    (pad 1 thru_hole rect (at 0 0) (size 3 3) (drill 1.52) (layers *.Cu *.Mask)
+    (pad 1 thru_hole rect (at 0 0 180) (size 3 3) (drill 1.52) (layers *.Cu *.Mask)
       (net 1 "Net-(12V-GND1-Pad1)"))
     (model ${KISYS3DMOD}/TerminalBlock.3dshapes/TerminalBlock_bornier-2_P5.08mm.wrl
@@
   )
   (module Connector_PinHeader_2.54mm:PinHeader_1x01_P2.54mm_Vertical (layer F.Cu)
-    (at 182.88 60.96 90)
+    (at 193.04 60.96 90)
     (descr "Through hole straight pin header, 1x01, 2.54mm pitch, single row")
     (tags "Through hole pin header THT 1x01 2.54mm single row")
@@
   )
   (module Connector_PinHeader_2.54mm:PinHeader_1x01_P2.54mm_Vertical (layer F.Cu)
-    (at 193.04 76.2 90)
+    (at 182.88 76.2 90)
     (descr "Through hole straight pin header, 1x01, 2.54mm pitch, single row")
     (tags "Through hole pin header THT 1x01 2.54mm single row")
@@
   )
   (module Connector_PinHeader_2.54mm:PinHeader_1x01_P2.54mm_Vertical (layer F.Cu)
-    (at 193.04 60.96 90)
+    (at 182.88 60.96 90)
     (descr "Through hole straight pin header, 1x01, 2.54mm pitch, single row")
     (tags "Through hole pin header THT 1x01 2.54mm single row")
@@
   )
   (module TerminalBlock:TerminalBlock_bornier-2_P5.08mm (layer F.Cu)
-    (at 167.64 91.44)
+    (at 172.72 91.44 180)
     (descr "simple 2-pin terminal block, pitch 5.08mm, revamped version of bornier2")
     (tags "terminal block bornier2")
@@
     (fp_line (start 7.79 4) (end 7.79 -4) (layer F.CrtYd) (width 0.05))
     (fp_line (start 7.79 4) (end -2.71 4) (layer F.CrtYd) (width 0.05))
-    (pad 1 thru_hole rect (at 0 0) (size 3 3) (drill 1.52) (layers *.Cu *.Mask)
+    (pad 1 thru_hole rect (at 0 0 180) (size 3 3) (drill 1.52) (layers *.Cu *.Mask)
       (net 8 ServoData))
-    (pad 2 thru_hole circle (at 5.08 0) (size 3 3) (drill 1.52) (layers *.Cu *.Mask)
+    (pad 2 thru_hole circle (at 5.08 0 180) (size 3 3) (drill 1.52) (layers *.Cu *.Mask)
       (net 14 GND))
     (model ${KISYS3DMOD}/TerminalBlock.3dshapes/TerminalBlock_bornier-2_P5.08mm.wrl
@@
     )
   )
-  (gr_text hemisphere-project.com (at 83.82 96.52) (layer F.SilkS)
-    (effects (font (size 1 1) (thickness 0.15)))
+  (gr_text "FAITES\nVOS\nJEUX !" (at 170.18 71.12) (layer F.SilkS)
+    (effects (font (size 1.5 1.5) (thickness 0.3)))
+  )
+  (gr_text hemisphere-project.com (at 88.9 99.06) (layer F.SilkS)
+    (effects (font (size 1.5 1.5) (thickness 0.25)))
   )
   (gr_text "(To Raspi)" (at 170.18 57.15) (layer F.SilkS)
@@
     (effects (font (size 1 1) (thickness 0.15)))
   )
-  (gr_text GND (at 172.72 86.36) (layer F.SilkS)
-    (effects (font (size 1 1) (thickness 0.15)))
-  )
-  (gr_text INPUT (at 190.5 83.82) (layer F.SilkS)
-    (effects (font (size 1 1) (thickness 0.15)))
-  )
-  (gr_text GND (at 193.04 86.36) (layer F.SilkS)
-    (effects (font (size 1 1) (thickness 0.15)))
-  )
-  (gr_text 12V (at 187.96 86.36) (layer F.SilkS)
-    (effects (font (size 1 1) (thickness 0.15)))
-  )
-  (gr_text Data (at 167.64 86.36) (layer F.SilkS)
+  (gr_text GND (at 167.64 96.52 180) (layer F.SilkS)
+    (effects (font (size 1 1) (thickness 0.15)))
+  )
+  (gr_text INPUT (at 190.5 99.06 180) (layer F.SilkS)
+    (effects (font (size 1 1) (thickness 0.15)))
+  )
+  (gr_text GND (at 187.96 96.52 180) (layer F.SilkS)
+    (effects (font (size 1 1) (thickness 0.15)))
+  )
+  (gr_text 12V (at 193.04 96.52 180) (layer F.SilkS)
+    (effects (font (size 1 1) (thickness 0.15)))
+  )
+  (gr_text Data (at 172.72 96.52 180) (layer F.SilkS)
     (effects (font (size 1 1) (thickness 0.15)))
   )
@@
     (arrow2b (pts (xy 63.5 35.56) (xy 64.626504 34.973579)))
   )
-  (gr_text SERVO (at 170.18 83.82) (layer F.SilkS)
+  (gr_text SERVO (at 170.18 99.06 180) (layer F.SilkS)
     (effects (font (size 1 1) (thickness 0.15)))
   )
@@
   (gr_line (start 198.12 43.18) (end 198.12 101.6) (layer Edge.Cuts) (width 0.05))
   (gr_line (start 63.5 43.18) (end 198.12 43.18) (layer Edge.Cuts) (width 0.05))
-  (segment (start 184.73 76.2) (end 182.88 76.2) (width 1) (layer B.Cu) (net 1) (status 20))
-  (segment (start 187.96 79.43) (end 184.73 76.2) (width 1) (layer B.Cu) (net 1))
-  (segment (start 187.96 91.44) (end 187.96 79.43) (width 1) (layer B.Cu) (net 1) (status 10))
-  (segment (start 193.04 91.44) (end 193.04 76.2) (width 1) (layer F.Cu) (net 2) (status 30))
+  (segment (start 193.04 91.44) (end 193.04 76.2) (width 1) (layer B.Cu) (net 1))
+  (segment (start 184.73 76.2) (end 182.88 76.2) (width 1) (layer B.Cu) (net 2))
+  (segment (start 187.96 79.43) (end 184.73 76.2) (width 1) (layer B.Cu) (net 2))
+  (segment (start 187.96 91.44) (end 187.96 79.43) (width 1) (layer B.Cu) (net 2))
   (segment (start 147.32 50.11) (end 147.32 48.26) (width 1) (layer B.Cu) (net 3) (status 20))
   (segment (start 158.17 60.96) (end 147.32 50.11) (width 1) (layer B.Cu) (net 3))
-  (segment (start 182.88 60.96) (end 158.17 60.96) (width 1) (layer B.Cu) (net 3) (status 10))
   (segment (start 101.6 96.52) (end 99.06 93.98) (width 1) (layer B.Cu) (net 3) (status 20))
   (segment (start 127 96.52) (end 101.6 96.52) (width 1) (layer B.Cu) (net 3))
@@
   (segment (start 158.17 60.96) (end 158.17 65.35) (width 1) (layer B.Cu) (net 3))
   (segment (start 147.32 49.36) (end 147.32 48.26) (width 0.25) (layer F.Cu) (net 3) (status 20))
+  (segment (start 190.5 65.35) (end 158.17 65.35) (width 1) (layer B.Cu) (net 3))
+  (segment (start 193.04 62.81) (end 190.5 65.35) (width 1) (layer B.Cu) (net 3))
+  (segment (start 193.04 60.96) (end 193.04 62.81) (width 1) (layer B.Cu) (net 3))
   (segment (start 97.96 48.26) (end 99.06 48.26) (width 0.25) (layer B.Cu) (net 4) (status 20))
   (segment (start 88.9 83.82) (end 86.36 83.82) (width 1) (layer B.Cu) (net 4) (status 10))
@@
   (segment (start 90.17 85.09) (end 99.06 76.2) (width 0.25) (layer F.Cu) (net 7) (status 20))
   (segment (start 75.730998 85.09) (end 90.17 85.09) (width 0.25) (layer F.Cu) (net 7))
-  (segment (start 166.37 90.17) (end 167.64 91.44) (width 0.25) (layer F.Cu) (net 8) (status 30))
-  (segment (start 161.049999 95.530001) (end 165.14 91.44) (width 1) (layer F.Cu) (net 8))
-  (segment (start 165.14 91.44) (end 167.64 91.44) (width 1) (layer F.Cu) (net 8) (status 20))
-  (segment (start 115.850001 95.530001) (end 161.049999 95.530001) (width 1) (layer F.Cu) (net 8))
-  (segment (start 99.06 78.74) (end 115.850001 95.530001) (width 1) (layer F.Cu) (net 8) (status 10))
+  (segment (start 173.99 92.71) (end 172.72 91.44) (width 0.25) (layer F.Cu) (net 8) (status 30))
+  (segment (start 172.72 93.94) (end 172.72 91.44) (width 1) (layer F.Cu) (net 8))
+  (segment (start 171.129999 95.530001) (end 172.72 93.94) (width 1) (layer F.Cu) (net 8))
+  (segment (start 115.850001 95.530001) (end 171.129999 95.530001) (width 1) (layer F.Cu) (net 8))
+  (segment (start 99.06 78.74) (end 115.850001 95.530001) (width 1) (layer F.Cu) (net 8))
   (segment (start 99.06 88.9) (end 106.68 96.52) (width 0.25) (layer F.Cu) (net 9) (status 10))
   (segment (start 106.68 96.52) (end 142.24 96.52) (width 0.25) (layer F.Cu) (net 9))
